Commit message: ready urdf + working sensors

File: src/mower_description/urdf/mower.urdf.xacro (robot description, xacro)
@@ -2,14 +2,16 @@
 <robot name="mower" xmlns:xacro="http://www.ros.org/wiki/xacro">
 <xacro:include filename="$(find mower_description)/urdf/realsense_camera.xacro"/>
+<xacro:include filename="$(find mower_description)/urdf/lidar.xacro"/>
 <xacro:arg name="robot_name" default="mower"/>
 <xacro:arg name="is_ignition" default="true"/>
-<!--<gazebo>
+<gazebo>
   <plugin filename="gz-sim-joint-state-publisher-system" name="gz::sim::systems::JointStatePublisher">
     <topic>/world/partitioned_world/model/robot/joint_state</topic>
     <joint_name>left_wheel_joint</joint_name>
     <joint_name>right_wheel_joint</joint_name>
+    <joint_name>caster_fork_joint</joint_name>
     <joint_name>caster_wheel_joint</joint_name>
   </plugin>
-</gazebo>-->
+</gazebo>
   <material name="gray">
     <color rgba="0.3 0.3 0.3 1.0"/>
@@ -174,5 +176,5 @@
 </collision>
   </link>
-  <!--<link name="imu_link">
+  <link name="imu_link">
     <visual>
       <geometry>
@@ -197,7 +199,7 @@
     <parent link="robot_base_link"/>
     <child link="imu_link"/>
-    <origin xyz="0.0 0.0 0.1" rpy="0 0 0"/>
-  </joint>-->
-<!--<xacro:rgbd_camera
+    <origin xyz="0.155 0.0 0.05" rpy="0 0 0"/>
+  </joint>
+<xacro:rgb_camera
     prefix="robot_camera_"
     camera_name="camera"
@@ -206,6 +208,14 @@
     xyz_offset="0.22 0 0.03"
     rpy_offset="0 0 0"
-  />-->
-<!--<gazebo reference="left_wheel">
+  />
+  <xacro:lidar_sensor
+    prefix="robot_lidar_"
+    parent="robot_base_link"
+    topic_name="/scan"
+    mesh_file="package://mower_description/meshes/rplidar_s2.stl"
+    xyz_offset="0.155 0 0.1"
+    rpy_offset="0 0 0"
+  />
+<gazebo reference="left_wheel">
   <mu1>1.0</mu1>
   <mu2>1.0</mu2>
@@ -225,9 +235,9 @@
   <kd>10.0</kd>
 </gazebo>
-<gazebo>
+<!--<gazebo>
   <plugin filename="gz_ros2_control-system" name="gz_ros2_control::GazeboSimROS2ControlPlugin">
     <parameters>$(find project_controller)/config/project_controllers.yaml</parameters>
   </plugin>
-</gazebo>
+</gazebo>-->
 <gazebo reference="imu_link">
 <sensor name="imu_sensor" type="imu">
@@ -258,4 +268,4 @@
     <state_interface name="velocity"/>
   </joint>
-</ros2_control>-->
+</ros2_control>
 </robot>

File: src/mower_description/urdf/realsense_camera.xacro (robot description, xacro)
@@ -2,5 +2,5 @@
 <robot xmlns:xacro="http://www.ros.org/wiki/xacro">
   <xacro:property name="M_PI" value="3.1415926535897931" />
-  <xacro:macro name="rgbd_camera" params="
+  <xacro:macro name="rgb_camera" params="
     prefix:=''
     camera_name:='camera'
@@ -17,12 +17,4 @@
     optical_xyz_offset:='0 0 0'
     optical_rpy_offset:='${-M_PI/2} 0 ${-M_PI/2}'
-    depth_frame_xyz_offset:='0 0 0'
-    depth_frame_rpy_offset:='0 0 0'
-    infra1_xyz_offset:='0 0 0'
-    infra1_rpy_offset:='0 0 0'
-    infra2_xyz_offset:='0 -0.05 0'
-    infra2_rpy_offset:='0 0 0'
-    color_xyz_offset:='0 0.015 0'
-    color_rpy_offset:='0 0 0'
     cam_width:=0.090
     cam_height:=0.025
@@ -41,9 +33,10 @@
     image_height:=480
     clip_near:=0.05
-    clip_far:=1.5
+    clip_far:=10.0
     update_rate:=20
     always_on:=1
     visualize:=true
     enable_collision:=false">
+    <!-- Fizyczne ogniwo kamery (wizualizacja + kolizja) -->
     <link name="${prefix}${camera_name}_link">
       <visual>
@@ -76,52 +69,12 @@
       <origin xyz="${xyz_offset}" rpy="${rpy_offset}"/>
     </joint>
-    <joint name="${prefix}${camera_name}_depth_joint" type="fixed">
-      <origin xyz="${depth_frame_xyz_offset}" rpy="${depth_frame_rpy_offset}"/>
-      <parent link="${prefix}${camera_name}_link"/>
-      <child link="${prefix}${camera_name}_depth_frame" />
+    <!-- Ramka optyczna (zgodna ze standardem układow współrzędnych kamer w ROS) -->
+    <joint name="${prefix}${camera_name}_optical_joint" type="fixed">
+      <origin xyz="${optical_xyz_offset}" rpy="${optical_rpy_offset}" />
+      <parent link="${prefix}${camera_name}_link" />
+      <child link="${prefix}${camera_name}_optical_frame" />
     </joint>
-    <link name="${prefix}${camera_name}_depth_frame"/>
-    <joint name="${prefix}${camera_name}_depth_optical_joint" type="fixed">
-      <origin xyz="${optical_xyz_offset}" rpy="${optical_rpy_offset}" />
-      <parent link="${prefix}${camera_name}_depth_frame" />
-      <child link="${prefix}${camera_name}_depth_optical_frame" />
-    </joint>
-    <link name="${prefix}${camera_name}_depth_optical_frame"/>
-    <joint name="${prefix}${camera_name}_infra1_joint" type="fixed">
-      <origin xyz="${infra1_xyz_offset}" rpy="${infra1_rpy_offset}" />
-      <parent link="${prefix}${camera_name}_link" />
-      <child link="${prefix}${camera_name}_infra1_frame" />
-    </joint>
-    <link name="${prefix}${camera_name}_infra1_frame"/>
-    <joint name="${prefix}${camera_name}_infra1_optical_joint" type="fixed">
-      <origin xyz="${optical_xyz_offset}" rpy="${optical_rpy_offset}" />
-      <parent link="${prefix}${camera_name}_infra1_frame" />
-      <child link="${prefix}${camera_name}_infra1_optical_frame" />
-    </joint>
-    <link name="${prefix}${camera_name}_infra1_optical_frame"/>
-    <joint name="${prefix}${camera_name}_infra2_joint" type="fixed">
-      <origin xyz="${infra2_xyz_offset}" rpy="${infra2_rpy_offset}" />
-      <parent link="${prefix}${camera_name}_link" />
-      <child link="${prefix}${camera_name}_infra2_frame" />
-    </joint>
-    <link name="${prefix}${camera_name}_infra2_frame"/>
-    <joint name="${prefix}${camera_name}_infra2_optical_joint" type="fixed">
-      <origin xyz="${optical_xyz_offset}" rpy="${optical_rpy_offset}" />
-      <parent link="${prefix}${camera_name}_infra2_frame" />
-      <child link="${prefix}${camera_name}_infra2_optical_frame" />
-    </joint>
-    <link name="${prefix}${camera_name}_infra2_optical_frame"/>
-    <joint name="${prefix}${camera_name}_color_joint" type="fixed">
-      <origin xyz="${color_xyz_offset}" rpy="${color_rpy_offset}" />
-      <parent link="${prefix}${camera_name}_link" />
-      <child link="${prefix}${camera_name}_color_frame" />
-    </joint>
-    <link name="${prefix}${camera_name}_color_frame"/>
-    <joint name="${prefix}${camera_name}_color_optical_joint" type="fixed">
-      <origin xyz="${optical_xyz_offset}" rpy="${optical_rpy_offset}" />
-      <parent link="${prefix}${camera_name}_color_frame" />
-      <child link="${prefix}${camera_name}_color_optical_frame" />
-    </joint>
-    <link name="${prefix}${camera_name}_color_optical_frame"/>
+    <link name="${prefix}${camera_name}_optical_frame"/>
+    <!-- Konfiguracja czujnika 2D w Gazebo -->
     <gazebo reference="${prefix}${camera_name}_link">
       <sensor name="${prefix}${camera_name}" type="camera">
@@ -133,7 +86,4 @@
             <format>R8G8B8</format>
           </image>
-          <depth_camera>
-            <output_format>L8</output_format>
-          </depth_camera>
           <clip>
             <near>${clip_near}</near>
@@ -144,6 +94,6 @@
         <update_rate>${update_rate}</update_rate>
         <visualize>${visualize}</visualize>
-        <topic>${camera_name}</topic>
-        <gz_frame_id>${prefix}${camera_name}_color_optical_frame</gz_frame_id>
+        <topic>${camera_name}/image_raw</topic>
+        <gz_frame_id>${prefix}${camera_name}_optical_frame</gz_frame_id>
       </sensor>
     </gazebo>

Commit message: added ekf to local localization and safety node

File: src/mower_description/urdf/mower.urdf.xacro (robot description, xacro)
@@ -51,5 +51,5 @@
     <parent link="base_link"/>
     <child link="robot_base_link"/>
-    <origin xyz="0.15 0 0.005" rpy="0 0 3.14159265"/>
+    <origin xyz="0.0 0 0.0" rpy="0 0 0"/>
 </joint>
   <link name="left_wheel">
